File: 15VBUCK.kicad_sch (KiCad schematic)
At the start: 11 parts, among them U3 LM76005RNPR

Commit message: Add complete layout-ready project files
Parts:
- removed Cout: 150.0μ, symbol Device:C_Polarized_US
- added Cout_15V1: 150u, BulkCapacitor_100u:CAP_EEFK_F_PAN, symbol BulkCap_150u:EEE-FP1V151AP
- Cboot_15V1: renamed from Cboot; value 470.0n -> 470n; footprint (none) -> Capacitor_SMD:C_0805_2012Metric
- Cin_15V1: renamed from C4; value 10µ -> 10u; footprint (none) -> Capacitor_SMD:C_0805_2012Metric
- Cinx_15V1: renamed from Cinx; value 470.0n -> 470n; footprint (none) -> Capacitor_SMD:C_0805_2012Metric
- Coutx_15V1: renamed from Coutx; value 470.0n -> 470n; footprint (none) -> Capacitor_SMD:C_0805_2012Metric
- Cvcc_15V1: renamed from Cvcc; value 2.2μ -> 2.2u; footprint (none) -> Capacitor_SMD:C_0603_1608Metric
- L1_15V1: renamed from L1; value 8.2μ -> 8.2u; footprint (none) -> Inductor_SMD:L_Bourns_SRP7028A_7.3x6.6mm
- Rfbb_15V1: renamed from Rfbb; footprint (none) -> Resistor_SMD:R_0603_1608Metric
- Rfbt_15V1: renamed from Rfbt; value 100.0k -> 100k; footprint (none) -> Resistor_SMD:R_0603_1608Metric
- Rpgood_15V1: renamed from Rpgood; value 100.0k -> 100k; footprint (none) -> Resistor_SMD:R_0603_1608Metric
- U5: renamed from U3; footprint RNP0030A -> Regulator:RNP0030A
Connections:
- net +15V: now also Cout_15V1.1
- net GND: now also Cout_15V1.2
- no-connect marks 0 -> 2
