File: PDB.kicad_sch (KiCad schematic)
At the start: 0 parts

Commit message: Add complete layout-ready project files
Parts:
- added A1: RaspberryPi_Pico, Module:RaspberryPi_Pico_Common_THT, symbol MCU_Module:RaspberryPi_Pico
- added J1: Conn_01x08_Socket, Connector_JST:JST_XH_B8B-XH-AM_1x08_P2.50mm_Vertical, symbol Connector:Conn_01x08_Socket
- added J2: Conn_01x02_Socket, Connector_AMASS:AMASS_XT30U-M_1x02_P5.0mm_Vertical, symbol Connector:Conn_01x02_Socket
- added J3, J6, J7: Conn_01x02_Socket, Connector_AMASS:AMASS_XT30U-F_1x02_P5.0mm_Vertical, symbol Connector:Conn_01x02_Socket
- added J5: Conn_01x02, symbol Connector_Generic:Conn_01x02
- added LDO_Cin1, LDO_Cout1: 10u, Capacitor_SMD:C_0805_2012Metric, symbol Device:C
- added Q1: IRF540N, Package_TO_SOT_THT:TO-220-3_Vertical, symbol Transistor_FET:IRF540N
- added U1: NCP1117-3.3_SOT223, Package_TO_SOT_SMD:SOT-223-3_TabPin2, symbol Regulator_Linear:NCP1117-3.3_SOT223
- added U2: PC817, Package_DIP:DIP-4_W7.62mm, symbol Isolator:PC817
Connections:
- net +20V: now also J5.1 (Pin_1)
- net GND: now also J5.2 (Pin_2), J6.2 (Pin_2), J7.2 (Pin_2), LDO_Cin1.2, LDO_Cout1.2, U1.1 (GND)
- new net: J3.2 (Pin_2), Q1.3 (S)
- new net: A1.13 (GND), A1.18 (GND), A1.23 (GND), A1.28 (GND), A1.3 (GND), A1.38 (GND), A1.8 (GND)
- new net: Q1.1 (G), U2.3
- new net +12V: J6.1 (Pin_1)
- new net +12V_3S: J2.1 (Pin_1), J3.1 (Pin_1), U2.4
- new net +15V: J7.1 (Pin_1)
- new net +3.3V: A1.36 (3V3), A1.37 (3V3_EN), LDO_Cout1.1, U1.2 (VO)
- new net +5V: LDO_Cin1.1, U1.3 (VI)
- new net GND_3S: J2.2 (Pin_2), Q1.2 (D)
- new net Opto_In+: A1.21 (GPIO16), U2.1
- new net Opto_In-: A1.22 (GPIO17), U2.2
